Commit message: ros_control launches simulation

File: ddbot_description/urdf/robot.urdf (robot description, URDF)
Before this commit: robot ddbot, 3 links, 2 joints
Joints:
- removed joint base_to_left_wheel
- removed joint base_to_right_wheel
- added joint wheel_left_joint: type continuous, parent base_link, child left_wheel, origin xyz=0 0.103 0, axis 0 1 0
- added joint wheel_right_joint: type continuous, parent base_link, child right_wheel, origin xyz=0 -0.103 0, axis 0 1 0

Commit message: simulation kinds of works but changes on lanch files are needed

File: ddbot_description/urdf/robot.urdf (robot description, URDF)
Before this commit: robot ddbot, 3 links, 2 joints
Joints:
- joint wheel_left_joint: origin xyz=0 0.103 0 -> xyz=0 0.111 0
- joint wheel_right_joint: origin xyz=0 -0.103 0 -> xyz=0 -0.111 0

Commit message: load stl error removed but stl still not displayed

File: ddbot_description/urdf/robot.urdf (robot description, URDF)
Before this commit: robot ddbot, 3 links, 2 joints
Links:
- link base_link: geometry collision box size=0.251 0.189 0.045; visual mesh filename=package://ddbot_description/meshes/body.stl scale=0.001 0.001 0.001
- link left_wheel: geometry collision cylinder length=0.016 radius=0.0254; visual mesh filename=package://ddbot_description/meshes/wheel.stl scale=0.001 0.001 0.001
- link right_wheel: geometry collision cylinder length=0.016 radius=0.0254; visual mesh filename=package://ddbot_description/meshes/wheel.stl scale=0.001 0.001 0.001

Commit message: gazebo and rviz works for simulation (without lidar)

File: ddbot_description/urdf/robot.urdf (robot description, URDF)
Before this commit: robot ddbot, 3 links, 2 joints
Links:
- link base_link: geometry collision mesh filename=package://ddbot_description/meshes/body.stl scale=0.001 0.001 0.001; visual mesh filename=package://ddbot_description/meshes/body.stl scale=0.001 0.001 0.001
Joints:
- joint wheel_left_joint: origin xyz=0 0.111 0 -> xyz=0 0.111 0.0254
- joint wheel_right_joint: origin xyz=0 -0.111 0 -> xyz=0 -0.111 0.0254
